File: emi-sombrero.kicad_sch (KiCad schematic)
At the start: 36 parts, among them J1 WE_687130149022, J2 Conn_02x20_Odd_Even, U1 74LVC1G29, U10 74LVC1G125, U8 ISO7761DBQ, U9 ISO7761DBQ, X1 SIT8008BC-83-33E-7.372800

Commit message: Add more testpoints, make DRDY optionally open collector.
Parts:
- added C40: 100n, Capacitor_SMD:C_0603_1608Metric, symbol Device:C_Small
- added R24: DNP, Resistor_SMD:R_0603_1608Metric, symbol Device:R_Small
- added R25: 10k, Resistor_SMD:R_0603_1608Metric, symbol Device:R_Small
- added TP21, TP22, TP23, TP24, TP25, TP26, TP27, TP28, TP29, TP30, TP31, TP32, TP33, TP36, TP37, TP38, TP39: TestPoint_Small, TestPoint:TestPoint_Pad_1.5x1.5mm, symbol Connector:TestPoint_Small
- added U11: 74LVC1G125, Package_TO_SOT_SMD:SOT-23-5, symbol 74xGxx:74LVC1G125
Connections:
- net CIPO: now also TP26.1
- net CLK: now also TP27.1
- net COPI: now also TP22.1
- net CS_A0: now also TP24.1
- net CS_A1: now also TP25.1
- net DRDY: now also TP30.1
- net DRDY_RPI: now also R24.2, R25.1, U11.4; no longer U9.7 (OUTF)
- net GND: now also C40.2, TP36.1, TP37.1, U11.2, U11.3 (GND)
- net SCK: now also TP21.1
- net START: now also TP29.1
- net VBUS: now also TP39.1
- net VCC: now also C40.1, R25.2, TP38.1, U11.5 (VCC)
- net ~{CS1}: now also TP31.1
- net ~{CS2}: now also TP32.1
- net ~{CS3}: now also TP33.1
- net ~{CS}: now also TP23.1
- net ~{RESET}: now also TP28.1
- new net: R24.1, U11.1, U9.7 (OUTF)
Other:
- moved on the sheet: C1, C39, R15, R16, R17, R18, R2, R3, R4, U1, X1
